File: teabiscuits_adc_4ch/teabiscuits_adc_4ch.sch (KiCad schematic (older format))
At the start: 83 parts, among them J1 Conn_Coaxial, J2 Conn_Coaxial, J3 Conn_Coaxial, J4 Conn_Coaxial, J5 Conn_Coaxial, J6 Conn_01x28, U1 ADAR7251, Y1 Crystal

Commit message: Misc updates
Parts:
- C23, C24: value C -> 16pF
- U1: symbol ADAR7251:ADAR7251 -> teabiscuits_adc_4ch-rescue:ADAR7251-ADAR7251
- Y1: value Crystal -> CX3225SB19200D0FPLCC
Changed lines of the file:
@@
 $EndDescr
 $Comp
-L ADAR7251:ADAR7251 U1
+L teabiscuits_adc_4ch-rescue:ADAR7251-ADAR7251 U1
 U 3 1 5EF69449
 P 2750 5550
@@
 $EndComp
 $Comp
-L ADAR7251:ADAR7251 U1
+L teabiscuits_adc_4ch-rescue:ADAR7251-ADAR7251 U1
 U 4 1 5EF6A4BC
 P 10000 4200
@@
 	3450 1850 2900 1850
 $Comp
-L ADAR7251:ADAR7251 U1
+L teabiscuits_adc_4ch-rescue:ADAR7251-ADAR7251 U1
 U 1 1 5EF67E81
 P 3550 750
@@
 P 9100 4500
 F 0 "Y1" V 9054 4631 50  0000 L CNN
-F 1 "Crystal" V 8900 4500 50  0000 L CNN
+F 1 "CX3225SB19200D0FPLCC" V 8900 4500 50  0000 L CNN
 F 2 "Crystal:Crystal_SMD_3225-4Pin_3.2x2.5mm" H 9100 4500 50  0001 C CNN
 F 3 "~" H 9100 4500 50  0001 C CNN
@@
 P 8950 4350
 F 0 "C23" V 8698 4350 50  0000 C CNN
-F 1 "C" V 8789 4350 50  0000 C CNN
+F 1 "16pF" V 8789 4350 50  0000 C CNN
 F 2 "Capacitor_SMD:C_0603_1608Metric" H 8988 4200 50  0001 C CNN
 F 3 "~" H 8950 4350 50  0001 C CNN
@@
 P 8950 4650
 F 0 "C24" V 8698 4650 50  0000 C CNN
-F 1 "C" V 8789 4650 50  0000 C CNN
+F 1 "16pF" V 8789 4650 50  0000 C CNN
 F 2 "Capacitor_SMD:C_0603_1608Metric" H 8988 4500 50  0001 C CNN
 F 3 "~" H 8950 4650 50  0001 C CNN
@@
 Connection ~ 9800 850
 $Comp
-L ADAR7251:ADAR7251 U1
+L teabiscuits_adc_4ch-rescue:ADAR7251-ADAR7251 U1
 U 2 1 5EF68A4E
 P 9900 750
