File: teabiscuits_compute/teabiscuits_compute.sch (KiCad schematic (older format))
At the start: 40 parts, among them J1 Conn_01x07, J10 Conn_Coaxial, J11 Conn_Coaxial, J2 Conn_01x07, J3 Conn_01x05, J4 Conn_01x03, J5 Conn_02x15_Counter_Clockwise, J7 Conn_Coaxial, J8 Conn_Coaxial, J9 Conn_Coaxial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

Commit message: Fixes to compute board
Connections:
- net +5V: now also U2.7 (V+), U3.7 (V+), U4.7 (V+), U5.7 (V+), U6.7 (V+); no longer U2.4 (V-), U3.4 (V-), U4.4 (V-), U5.4 (V-), U6.4 (V-)
- net -5V: now also U2.4 (V-), U3.4 (V-), U4.4 (V-), U5.4 (V-), U6.4 (V-); no longer U2.7 (V+), U3.7 (V+), U4.7 (V+), U5.7 (V+), U6.7 (V+)
Changed lines of the file:
@@
 L power:+5V #PWR047
 U 1 1 5F0CAE55
+P 10500 750
+F 0 "#PWR047" H 10500 600 50  0001 C CNN
+F 1 "+5V" H 10515 923 50  0000 C CNN
+F 2 "" H 10500 750 50  0001 C CNN
+F 3 "" H 10500 750 50  0001 C CNN
+	1    10500 750
+	1    0    0    -1
+$EndComp
+$Comp
+L power:-5V #PWR046
+U 1 1 5F0C6FEE
 P 10500 1350
-F 0 "#PWR047" H 10500 1200 50  0001 C CNN
-F 1 "+5V" H 10515 1523 50  0000 C CNN
+F 0 "#PWR046" H 10500 1450 50  0001 C CNN
+F 1 "-5V" H 10515 1523 50  0000 C CNN
 F 2 "" H 10500 1350 50  0001 C CNN
 F 3 "" H 10500 1350 50  0001 C CNN
 	1    10500 1350
 	-1   0    0    1
-$EndComp
-$Comp
-L power:-5V #PWR046
-U 1 1 5F0C6FEE
-P 10500 750
-F 0 "#PWR046" H 10500 850 50  0001 C CNN
-F 1 "-5V" H 10515 923 50  0000 C CNN
-F 2 "" H 10500 750 50  0001 C CNN
-F 3 "" H 10500 750 50  0001 C CNN
-	1    10500 750
-	1    0    0    -1
 $EndComp
 $Comp
@@
 L power:+5V #PWR049
 U 1 1 5F143739
+P 10500 1950
+F 0 "#PWR049" H 10500 1800 50  0001 C CNN
+F 1 "+5V" H 10515 2123 50  0000 C CNN
+F 2 "" H 10500 1950 50  0001 C CNN
+F 3 "" H 10500 1950 50  0001 C CNN
+	1    10500 1950
+	1    0    0    -1
+$EndComp
+$Comp
+L power:-5V #PWR048
+U 1 1 5F143743
 P 10500 2550
-F 0 "#PWR049" H 10500 2400 50  0001 C CNN
-F 1 "+5V" H 10515 2723 50  0000 C CNN
+F 0 "#PWR048" H 10500 2650 50  0001 C CNN
+F 1 "-5V" H 10515 2723 50  0000 C CNN
 F 2 "" H 10500 2550 50  0001 C CNN
 F 3 "" H 10500 2550 50  0001 C CNN
 	1    10500 2550
 	-1   0    0    1
-$EndComp
-$Comp
-L power:-5V #PWR048
-U 1 1 5F143743
-P 10500 1950
-F 0 "#PWR048" H 10500 2050 50  0001 C CNN
-F 1 "-5V" H 10515 2123 50  0000 C CNN
-F 2 "" H 10500 1950 50  0001 C CNN
-F 3 "" H 10500 1950 50  0001 C CNN
-	1    10500 1950
-	1    0    0    -1
 $EndComp
 $Comp
@@
 L power:+5V #PWR051
 U 1 1 5F177FE7
+P 10500 3300
+F 0 "#PWR051" H 10500 3150 50  0001 C CNN
+F 1 "+5V" H 10515 3473 50  0000 C CNN
+F 2 "" H 10500 3300 50  0001 C CNN
+F 3 "" H 10500 3300 50  0001 C CNN
+	1    10500 3300
+	1    0    0    -1
+$EndComp
+$Comp
+L power:-5V #PWR050
+U 1 1 5F177FF1
 P 10500 3900
-F 0 "#PWR051" H 10500 3750 50  0001 C CNN
-F 1 "+5V" H 10515 4073 50  0000 C CNN
+F 0 "#PWR050" H 10500 4000 50  0001 C CNN
+F 1 "-5V" H 10515 4073 50  0000 C CNN
 F 2 "" H 10500 3900 50  0001 C CNN
 F 3 "" H 10500 3900 50  0001 C CNN
 	1    10500 3900
 	-1   0    0    1
-$EndComp
-$Comp
-L power:-5V #PWR050
-U 1 1 5F177FF1
-P 10500 3300
-F 0 "#PWR050" H 10500 3400 50  0001 C CNN
-F 1 "-5V" H 10515 3473 50  0000 C CNN
-F 2 "" H 10500 3300 50  0001 C CNN
-F 3 "" H 10500 3300 50  0001 C CNN
-	1    10500 3300
-	1    0    0    -1
 $EndComp
 $Comp
@@
 L power:+5V #PWR053
 U 1 1 5F17803F
+P 10500 4500
+F 0 "#PWR053" H 10500 4350 50  0001 C CNN
+F 1 "+5V" H 10515 4673 50  0000 C CNN
+F 2 "" H 10500 4500 50  0001 C CNN
+F 3 "" H 10500 4500 50  0001 C CNN
+	1    10500 4500
+	1    0    0    -1
+$EndComp
+$Comp
+L power:-5V #PWR052
+U 1 1 5F178049
 P 10500 5100
-F 0 "#PWR053" H 10500 4950 50  0001 C CNN
-F 1 "+5V" H 10515 5273 50  0000 C CNN
+F 0 "#PWR052" H 10500 5200 50  0001 C CNN
+F 1 "-5V" H 10515 5273 50  0000 C CNN
 F 2 "" H 10500 5100 50  0001 C CNN
 F 3 "" H 10500 5100 50  0001 C CNN
 	1    10500 5100
 	-1   0    0    1
-$EndComp
-$Comp
-L power:-5V #PWR052
-U 1 1 5F178049
-P 10500 4500
-F 0 "#PWR052" H 10500 4600 50  0001 C CNN
-F 1 "-5V" H 10515 4673 50  0000 C CNN
-F 2 "" H 10500 4500 50  0001 C CNN
-F 3 "" H 10500 4500 50  0001 C CNN
-	1    10500 4500
-	1    0    0    -1
 $EndComp
 $Comp
@@
 L power:+5V #PWR022
 U 1 1 5F1C841C
+P 7850 750
+F 0 "#PWR022" H 7850 600 50  0001 C CNN
+F 1 "+5V" H 7865 923 50  0000 C CNN
+F 2 "" H 7850 750 50  0001 C CNN
+F 3 "" H 7850 750 50  0001 C CNN
+	1    7850 750
+	1    0    0    -1
+$EndComp
+$Comp
+L power:-5V #PWR021
+U 1 1 5F1C8426
 P 7850 1350
-F 0 "#PWR022" H 7850 1200 50  0001 C CNN
-F 1 "+5V" H 7865 1523 50  0000 C CNN
+F 0 "#PWR021" H 7850 1450 50  0001 C CNN
+F 1 "-5V" H 7865 1523 50  0000 C CNN
 F 2 "" H 7850 1350 50  0001 C CNN
 F 3 "" H 7850 1350 50  0001 C CNN
@@
 $EndComp
 $Comp
-L power:-5V #PWR021
-U 1 1 5F1C8426
-P 7850 750
-F 0 "#PWR021" H 7850 850 50  0001 C CNN
-F 1 "-5V" H 7865 923 50  0000 C CNN
-F 2 "" H 7850 750 50  0001 C CNN
-F 3 "" H 7850 750 50  0001 C CNN
-	1    7850 750
-	1    0    0    -1
-$EndComp
-$Comp
