File: teabiscuits_integrated/teabiscuits_compute.kicad_pcb (KiCad board)
At the start: 2 copper layers, 122.8 x 71.8 mm, 38 parts, among them J1 Barrel_Jack, J10 Conn_Coaxial, J2 Conn_02x04_Odd_Even, J3 Conn_01x03, J4 Conn_01x03, J5 Conn_02x03_Odd_Even, J6 J1B1211CCD, J7 Conn_Coaxial, J8 Conn_Coaxial, J9 Conn_01x03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

Commit message: r4 of integrated pcb
Parts:
- added J11: Conn_02x04_Odd_Even, Connector_PinHeader_2.54mm:PinHeader_2x04_P2.54mm_Vertical, F.Cu at (175.7, 104.8)
- J2: moved to B.Cu
- moved J1 12.0 mm to (201.0, 156.0), turned to 0 degrees
- moved J2 8.95 mm to (175.7, 120.2)
- moved U1 7.63 mm to (140.5, 134.6), turned to 90 degrees
- moved J5 0.25 mm to (128.0, 130.0)
Connections:
- net Net-(J5-Pad3) renamed LED
- C8 pad 1: Net-(C8-Pad1) -> GND
- J5 pad 4: Net-(C8-Pad1) -> GND
- J6 pad 1: T+ -> T-
- J6 pad 2: Net-(C8-Pad2) -> T+
- J6 pad 3: T- -> Net-(C8-Pad2)
- J6 pad 4: R+ -> Net-(J6-Pad4)
- J6 pad 5: Net-(C8-Pad2) -> Net-(J6-Pad5)
- J6 pad 6: R- -> Net-(J6-Pad6)
- J6 pad 7: Net-(J6-Pad7) -> R+
- J6 pad 8: Net-(C8-Pad1) -> R-
- J6 pad 9: Net-(C8-Pad1) -> GND
Routing:
- net Net-(C8-Pad1): track 56.2 -> 0.00 mm
- net 28: track 23.4 -> 67.8 mm
- net SPI4_MISO: track 32.5 -> 66.9 mm, vias 0 -> 2
- net SPI4_CS0: track 32.3 -> 65.9 mm
- net IOREF: track 73.7 -> 104.3 mm, vias 0 -> 1
- net O1: track 25.5 -> 45.6 mm
- net SPI4_SCLK: track 43.6 -> 62.2 mm
- net +5V: track 170.9 -> 186.8 mm, vias 4 -> 6
- net Net-(J1-Pad1): track 23.1 -> 8.38 mm
- net A1: track 37.1 -> 49.0 mm, vias 1 -> 2
- net -5V: track 118.2 -> 128.8 mm
- net GND: track 13.2 -> 20.3 mm, vias 4 -> 9
- net R+: track 55.1 -> 50.0 mm
- net T+: track 55.0 -> 50.0 mm
- net T-: track 54.6 -> 50.0 mm
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Other:
- board text added: "Teensy Integrated r4"
- board text removed: "T- T+"
- board text removed: "Teensy Integrated r1"
