File: teabiscuits_dac_mcp48/teabiscuits_dac_mcp48.kicad_pcb (KiCad board)
At the start: 2 copper layers, 50.5 x 14.5 mm, 13 parts, among them J2 Conn_01x10, U1 MCP4801, U2 OP07

Commit message: Updated DAC layout
Parts:
- renumbered Je to J1
Connections:
- U2 pad 2: Net-(R3-Pad1) -> Net-(R2-Pad1)
- U2 pad 3: Net-(R2-Pad1) -> Net-(R3-Pad1)
Routing:
- net Net-(R3-Pad1): track 9.45 -> 6.39 mm, vias 2 -> 0
- net Net-(R2-Pad1): track 13.5 -> 15.5 mm
Other:
- board text added: "DAC MCP48 r2"
- board text removed: "ADC MCP48 r1"

Commit message: MCP48 DAC r3
Parts:
- R2, R4, R5: value R -> 1K
Connections:
- R5 pad 2: Net-(R2-Pad1) -> Net-(R3-Pad1)
- U2 pad 2: Net-(R2-Pad1) -> Net-(R3-Pad1)
- U2 pad 3: Net-(R3-Pad1) -> Net-(R2-Pad1)
Routing:
- net Net-(R2-Pad1): track 15.5 -> 7.37 mm
- net Net-(R3-Pad1): track 6.39 -> 12.7 mm
Other:
- board text added: "DAC MCP48 r3"
- board text removed: "DAC MCP48 r2"
