File: teabiscuits_dac_mcp48/teabiscuits_dac_mcp48.sch (KiCad schematic (older format))
At the start: 13 parts, among them J1 Conn_Coaxial, J2 Conn_01x10, U1 MCP4801, U2 OP07

Commit message: Updated DAC layout
Connections:
- net at R3.1, R4.2: now also U2.3 (+); no longer U2.2 (-)
- net at R2.1, R5.2: now also U2.2 (-); no longer U2.3 (+)
Changed lines of the file:
@@
 F 3 "https://www.analog.com/media/en/technical-documentation/data-sheets/OP07.pdf" H 7850 3750 50  0001 C CNN
 	1    7800 3600
-	1    0    0    -1
+	1    0    0    1
 $EndComp
 $Comp
@@
 L power:+5V #PWR06
 U 1 1 5F5B996D
-P 7700 3300
-F 0 "#PWR06" H 7700 3150 50  0001 C CNN
-F 1 "+5V" H 7715 3473 50  0000 C CNN
-F 2 "" H 7700 3300 50  0001 C CNN
-F 3 "" H 7700 3300 50  0001 C CNN
-	1    7700 3300
-	1    0    0    -1
-$EndComp
-$Comp
-L power:-5V #PWR07
-U 1 1 5F5B9FBF
 P 7700 3900
-F 0 "#PWR07" H 7700 4000 50  0001 C CNN
-F 1 "-5V" H 7715 4073 50  0000 C CNN
+F 0 "#PWR06" H 7700 3750 50  0001 C CNN
+F 1 "+5V" H 7715 4073 50  0000 C CNN
 F 2 "" H 7700 3900 50  0001 C CNN
 F 3 "" H 7700 3900 50  0001 C CNN
 	1    7700 3900
 	-1   0    0    1
+$EndComp
+$Comp
+L power:-5V #PWR07
+U 1 1 5F5B9FBF
+P 7700 3300
+F 0 "#PWR07" H 7700 3400 50  0001 C CNN
+F 1 "-5V" H 7715 3473 50  0000 C CNN
+F 2 "" H 7700 3300 50  0001 C CNN
+F 3 "" H 7700 3300 50  0001 C CNN
+	1    7700 3300
+	1    0    0    -1
 $EndComp
 $Comp
@@
 Wire Wire Line
 	8450 3600 8100 3600
-Connection ~ 8100 3600
 $Comp
 L power:GND #PWR08
@@
 	1    0    0    -1
 $EndComp
+Connection ~ 8100 3600
 $EndSCHEMATC

Commit message: MCP48 DAC r3
Parts:
- R2, R4, R5: value R -> 1K
Connections:
- net at R5.2, U2.2 (-): now also R3.1, R4.2; no longer R2.1
- new net: R2.1, U2.3 (+)
Other:
- moved on the sheet: C1, C2, R1, R2, R3, R4, U1
Changed lines of the file:
@@
 L Analog_DAC:MCP4801 U1
 U 1 1 5F5AF9E7
-P 5500 3500
-F 0 "U1" H 5100 3850 50  0000 L CNN
-F 1 "MCP4801" H 5400 3500 50  0000 L CNN
-F 2 "Package_SO:SOIC-8_3.9x4.9mm_P1.27mm" H 6400 3400 50  0001 C CNN
-F 3 "http://ww1.microchip.com/downloads/en/DeviceDoc/22244B.pdf" H 6400 3400 50  0001 C CNN
-	1    5500 3500
+P 5650 3700
+F 0 "U1" H 5250 4050 50  0000 L CNN
+F 1 "MCP4801" H 5550 3700 50  0000 L CNN
+F 2 "Package_SO:SOIC-8_3.9x4.9mm_P1.27mm" H 6550 3600 50  0001 C CNN
+F 3 "http://ww1.microchip.com/downloads/en/DeviceDoc/22244B.pdf" H 6550 3600 50  0001 C CNN
+	1    5650 3700
 	1    0    0    -1
 $EndComp
@@
 L power:GND #PWR03
 U 1 1 5F5B1060
-P 5500 3900
-F 0 "#PWR03" H 5500 3650 50  0001 C CNN
-F 1 "GND" H 5505 3727 50  0000 C CNN
-F 2 "" H 5500 3900 50  0001 C CNN
-F 3 "" H 5500 3900 50  0001 C CNN
-	1    5500 3900
+P 5650 4100
+F 0 "#PWR03" H 5650 3850 50  0001 C CNN
+F 1 "GND" H 5655 3927 50  0000 C CNN
+F 2 "" H 5650 4100 50  0001 C CNN
+F 3 "" H 5650 4100 50  0001 C CNN
+	1    5650 4100
 	1    0    0    -1
 $EndComp
@@
 L power:+3.3V #PWR02
 U 1 1 5F5B35BE
-P 5500 2400
-F 0 "#PWR02" H 5500 2250 50  0001 C CNN
-F 1 "+3.3V" H 5515 2573 50  0000 C CNN
-F 2 "" H 5500 2400 50  0001 C CNN
-F 3 "" H 5500 2400 50  0001 C CNN
-	1    5500 2400
-	1    0    0    -1
-$EndComp
-Wire Wire Line
-	5500 3100 5500 3050
+P 5650 2600
+F 0 "#PWR02" H 5650 2450 50  0001 C CNN
+F 1 "+3.3V" H 5665 2773 50  0000 C CNN
+F 2 "" H 5650 2600 50  0001 C CNN
+F 3 "" H 5650 2600 50  0001 C CNN
+	1    5650 2600
+	1    0    0    -1
+$EndComp
+Wire Wire Line
+	5650 3300 5650 3250
 $Comp
 L Device:C C2
 U 1 1 5F5B4078
-P 5650 3050
-F 0 "C2" V 5398 3050 50  0000 C CNN
-F 1 "C" V 5489 3050 50  0000 C CNN
-F 2 "Capacitor_SMD:C_1206_3216Metric" H 5688 2900 50  0001 C CNN
-F 3 "~" H 5650 3050 50  0001 C CNN
-	1    5650 3050
-	0    1    1    0
-$EndComp
-Connection ~ 5500 3050
+P 5800 3250
+F 0 "C2" V 5548 3250 50  0000 C CNN
+F 1 "C" V 5639 3250 50  0000 C CNN
+F 2 "Capacitor_SMD:C_1206_3216Metric" H 5838 3100 50  0001 C CNN
+F 3 "~" H 5800 3250 50  0001 C CNN
+	1    5800 3250
+	0    1    1    0
+$EndComp
+Connection ~ 5650 3250
 $Comp
 L Device:CP C1
 U 1 1 5F5B4639
-P 5650 2600
-F 0 "C1" V 5905 2600 50  0000 C CNN
-F 1 "CP" V 5814 2600 50  0000 C CNN
-F 2 "Capacitor_Tantalum_SMD:CP_EIA-3216-18_Kemet-A" H 5688 2450 50  0001 C CNN
-F 3 "~" H 5650 2600 50  0001 C CNN
-	1    5650 2600
+P 5800 2800
+F 0 "C1" V 6055 2800 50  0000 C CNN
+F 1 "CP" V 5964 2800 50  0000 C CNN
+F 2 "Capacitor_Tantalum_SMD:CP_EIA-3216-18_Kemet-A" H 5838 2650 50  0001 C CNN
+F 3 "~" H 5800 2800 50  0001 C CNN
+	1    5800 2800
 	0    -1   -1   0
 $EndComp
 Wire Wire Line
-	5500 2400 5500 2600
-Connection ~ 5500 2600
-Wire Wire Line
-	5500 2600 5500 3050
-Wire Wire Line
-	5800 2600 5800 3050
+	5650 2600 5650 2800
+Connection ~ 5650 2800
+Wire Wire Line
+	5650 2800 5650 3250
+Wire Wire Line
+	5950 2800 5950 3250
 $Comp
 L power:GND #PWR04
 U 1 1 5F5B5D4F
-P 5800 3050
-F 0 "#PWR04" H 5800 2800 50  0001 C CNN
-F 1 "GND" H 5805 2877 50  0000 C CNN
-F 2 "" H 5800 3050 50  0001 C CNN
-F 3 "" H 5800 3050 50  0001 C CNN
-	1    5800 3050
-	1    0    0    -1
-$EndComp
-Connection ~ 5800 3050
+P 5950 3250
+F 0 "#PWR04" H 5950 3000 50  0001 C CNN
+F 1 "GND" H 5955 3077 50  0000 C CNN
+F 2 "" H 5950 3250 50  0001 C CNN
+F 3 "" H 5950 3250 50  0001 C CNN
+	1    5950 3250
+	1    0    0    -1
+$EndComp
+Connection ~ 5950 3250
 $Comp
 L Connector_Generic:Conn_01x10 J2
@@
 	1    0    0    -1
 $EndComp
-Text GLabel 5000 3600 0    50   Input ~ 0
+Text GLabel 5150 3800 0    50   Input ~ 0
 SCK
 Text GLabel 9200 2000 0    50   Input ~ 0
 SCK
-Text GLabel 5000 3700 0    50   Input ~ 0
+Text GLabel 5150 3900 0    50   Input ~ 0
 SDI
 Text GLabel 9200 2100 0    50   Input ~ 0
 SDI
-Text GLabel 5000 3500 0    50   Input ~ 0
+Text GLabel 5150 3700 0    50   Input ~ 0
 CS
 Text GLabel 9200 2300 0    50   Input ~ 0
 CS
-Text GLabel 5000 3400 0    50   Input ~ 0
+Text GLabel 5150 3600 0    50   Input ~ 0
 LDAC
 Text GLabel 9200 2900 0    50   Input ~ 0
@@
 	1    0    0    -1
 $EndComp
-$Comp
-L Device:R R1
-U 1 1 5F5BDA40
-P 4850 3150
-F 0 "R1" H 4920 3196 50  0000 L CNN
-F 1 "R" H 4920 3105 50  0000 L CNN
-F 2 "Resistor_SMD:R_1206_3216Metric" V 4780 3150 50  0001 C CNN
-F 3 "~" H 4850 3150 50  0001 C CNN
-	1    4850 3150
-	1    0    0    -1
-$EndComp
-Wire Wire Line
-	4850 3300 5000 3300
+Wire Wire Line
+	5000 3500 5150 3500
 $Comp
 L power:+3.3V #PWR01
 U 1 1 5F5BE428
-P 4850 3000
-F 0 "#PWR01" H 4850 2850 50  0001 C CNN
-F 1 "+3.3V" H 4865 3173 50  0000 C CNN
-F 2 "" H 4850 3000 50  0001 C CNN
-F 3 "" H 4850 3000 50  0001 C CNN
-	1    4850 3000
+P 5000 3200
+F 0 "#PWR01" H 5000 3050 50  0001 C CNN
+F 1 "+3.3V" H 5015 3373 50  0000 C CNN
+F 2 "" H 5000 3200 50  0001 C CNN
+F 3 "" H 5000 3200 50  0001 C CNN
+	1    5000 3200
 	1    0    0    -1
 $EndComp
 Text GLabel 9200 2800 0    50   Input ~ 0
 REF
-Text GLabel 7050 3700 0    50   Input ~ 0
+Text GLabel 6900 2950 0    50   Input ~ 0
 REF
-$Comp
-L Device:R R3
-U 1 1 5F5C00A5
-P 7200 3700
-F 0 "R3" V 7300 3700 50  0000 C CNN
-F 1 "R" V 7084 3700 50  0000 C CNN
-F 2 "Resistor_SMD:R_1206_3216Metric" V 7130 3700 50  0001 C CNN
-F 3 "~" H 7200 3700 50  0001 C CNN
-	1    7200 3700
-	0    1    1    0
-$EndComp
 $Comp
 L Device:R R4
 U 1 1 5F5C0CD1
-P 7350 3850
-F 0 "R4" H 7280 3804 50  0000 R CNN
-F 1 "R" H 7280 3895 50  0000 R CNN
-F 2 "Resistor_SMD:R_1206_3216Metric" V 7280 3850 50  0001 C CNN
-F 3 "~" H 7350 3850 50  0001 C CNN
-	1    7350 3850
+P 7200 3100
+F 0 "R4" H 7130 3054 50  0000 R CNN
+F 1 "1K" H 7130 3145 50  0000 R CNN
+F 2 "Resistor_SMD:R_1206_3216Metric" V 7130 3100 50  0001 C CNN
+F 3 "~" H 7200 3100 50  0001 C CNN
+	1    7200 3100
 	-1   0    0    1
 $EndComp
@@
 L power:GND #PWR05
 U 1 1 5F5C10CD
-P 7350 4000
-F 0 "#PWR05" H 7350 3750 50  0001 C CNN
-F 1 "GND" H 7355 3827 50  0000 C CNN
-F 2 "" H 7350 4000 50  0001 C CNN
-F 3 "" H 7350 4000 50  0001 C CNN
-	1    7350 4000
-	1    0    0    -1
-$EndComp
-Wire Wire Line
-	7350 3700 7500 3700
-Connection ~ 7350 3700
-$Comp
-L Device:R R2
-U 1 1 5F5C17B9
-P 6250 3500
-F 0 "R2" V 6350 3500 50  0000 C CNN
-F 1 "R" V 6134 3500 50  0000 C CNN
-F 2 "Resistor_SMD:R_1206_3216Metric" V 6180 3500 50  0001 C CNN
-F 3 "~" H 6250 3500 50  0001 C CNN
-	1    6250 3500
-	0    1    1    0
-$EndComp
+P 7200 3250
+F 0 "#PWR05" H 7200 3000 50  0001 C CNN
+F 1 "GND" H 7205 3077 50  0000 C CNN
+F 2 "" H 7200 3250 50  0001 C CNN
+F 3 "" H 7200 3250 50  0001 C CNN
+	1    7200 3250
+	1    0    0    -1
+$EndComp
+Wire Wire Line
+	7200 2950 7350 2950
+Connection ~ 7200 2950
 Wire Wire Line
 	7500 3500 7350 3500
-$Comp
-L Device:R R5
-U 1 1 5F5C2047
-P 7800 2950
-F 0 "R5" V 7593 2950 50  0000 C CNN
-F 1 "R" V 7684 2950 50  0000 C CNN
-F 2 "Resistor_SMD:R_1206_3216Metric" V 7730 2950 50  0001 C CNN
-F 3 "~" H 7800 2950 50  0001 C CNN
-	1    7800 2950
-	0    1    1    0
-$EndComp
 Wire Wire Line
 	7650 2950 7350 2950
 Wire Wire Line
 	7350 2950 7350 3500
-Connection ~ 7350 3500
-Wire Wire Line
-	7350 3500 6400 3500
 Wire Wire Line
 	7950 2950 8100 2950
@@
 $EndComp
 Connection ~ 8100 3600
+Wire Wire Line
+	7500 3700 6550 3700
+Connection ~ 7350 2950
+$Comp
+L Device:R R1
+U 1 1 5F5BDA40
+P 5000 3350
+F 0 "R1" H 5070 3396 50  0000 L CNN
+F 1 "R" H 5070 3305 50  0000 L CNN
+F 2 "Resistor_SMD:R_1206_3216Metric" V 4930 3350 50  0001 C CNN
+F 3 "~" H 5000 3350 50  0001 C CNN
+	1    5000 3350
+	1    0    0    -1
+$EndComp
+$Comp
+L Device:R R5
+U 1 1 5F5C2047
+P 7800 2950
+F 0 "R5" V 7593 2950 50  0000 C CNN
+F 1 "1K" V 7684 2950 50  0000 C CNN
+F 2 "Resistor_SMD:R_1206_3216Metric" V 7730 2950 50  0001 C CNN
+F 3 "~" H 7800 2950 50  0001 C CNN
+	1    7800 2950
+	0    1    1    0
+$EndComp
+$Comp
+L Device:R R2
+U 1 1 5F5C17B9
+P 6400 3700
+F 0 "R2" V 6500 3700 50  0000 C CNN
+F 1 "1K" V 6284 3700 50  0000 C CNN
+F 2 "Resistor_SMD:R_1206_3216Metric" V 6330 3700 50  0001 C CNN
+F 3 "~" H 6400 3700 50  0001 C CNN
+	1    6400 3700
+	0    1    1    0
+$EndComp
+$Comp
+L Device:R R3
+U 1 1 5F5C00A5
+P 7050 2950
+F 0 "R3" V 7150 2950 50  0000 C CNN
+F 1 "R" V 6934 2950 50  0000 C CNN
+F 2 "Resistor_SMD:R_1206_3216Metric" V 6980 2950 50  0001 C CNN
+F 3 "~" H 7050 2950 50  0001 C CNN
+	1    7050 2950
+	0    1    1    0
+$EndComp
 $EndSCHEMATC
