File: teabiscuits_integween/teabiscuits_compute.kicad_pcb (KiCad board)
At the start: 2 copper layers, 65.5 x 63.8 mm, 17 parts, among them J2 Conn_02x05_Odd_Even, J3 Conn_01x03, J4 Conn_02x05_Odd_Even, J5 Conn_02x03_Odd_Even, J6 J1B1211CCD, U1 teensy41, U2 PDME1-S5-D3-S, U3 ADP7142AUJZ-2.5, U4 ADP7182AUJZ-2.5, U5 REF5020AD

Commit message: integween r9
Connections:
- J2 pad 7: +5V -> +2V5
Routing:
- net +5V: track 103.0 -> 0.00 mm
- net +2V5: track 51.1 -> 106.3 mm, vias 0 -> 3
Other:
- board text added: "Teabiscuits Integween r9"
- board text removed: "Teabiscuits Integween r8"
Changed lines of the file:
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@@
     (thickness 1.6)
     (drawings 5)
-    (tracks 419)
+    (tracks 421)
     (zones 0)
     (modules 17)
@@
       (net 40 -2V5))
     (pad 7 thru_hole oval (at 0 -7.62 90) (size 1.7 1.7) (drill 1) (layers *.Cu *.Mask)
-      (net 1 +5V))
+      (net 39 +2V5))
     (pad 6 thru_hole oval (at 2.54 -5.08 90) (size 1.7 1.7) (drill 1) (layers *.Cu *.Mask)
       (net 42 IOREF))
@@
     )
   )
-  (gr_text "Teabiscuits Integween r8" (at 98.25 127.5 90) (layer F.SilkS)
+  (gr_text "Teabiscuits Integween r9" (at 98.25 127.5 90) (layer F.SilkS)
     (effects (font (size 1.5 1.5) (thickness 0.3)))
   )
@@
   (gr_line (start 93 169.5) (end 158.5 169.5) (layer Edge.Cuts) (width 0.05))
   (via (at 156.25 107.75) (size 2.2) (drill 2.1) (layers F.Cu B.Cu) (net 0))
-  (segment (start 118.63 168.5) (end 149 168.5) (width 0.5) (layer F.Cu) (net 1))
-  (segment (start 150.75 166.75) (end 150.75 164.25) (width 0.5) (layer F.Cu) (net 1))
-  (segment (start 149 168.5) (end 150.75 166.75) (width 0.5) (layer F.Cu) (net 1))
-  (segment (start 109 115.75) (end 106.75 113.5) (width 0.5) (layer B.Cu) (net 1))
-  (segment (start 113.67499 122.17499) (end 109 117.5) (width 0.5) (layer B.Cu) (net 1))
-  (segment (start 109 117.5) (end 109 115.75) (width 0.5) (layer B.Cu) (net 1))
-  (segment (start 113.67499 163.54499) (end 113.67499 122.17499) (width 0.5) (layer B.Cu) (net 1))
-  (segment (start 101.88 112.88) (end 102.5 113.5) (width 0.5) (layer B.Cu) (net 1))
-  (segment (start 101.88 110.25) (end 101.88 112.88) (width 0.5) (layer B.Cu) (net 1))
-  (segment (start 106.75 113.5) (end 102.5 113.5) (width 0.5) (layer B.Cu) (net 1))
-  (segment (start 118.63 168.5) (end 117 166.87) (width 0.5) (layer F.Cu) (net 1))
-  (segment (start 113.67499 163.54499) (end 117 166.87) (width 0.5) (layer B.Cu) (net 1))
   (via (at 95 107.75) (size 2.2) (drill 2.1) (layers F.Cu B.Cu) (net 2))
   (via (at 156.25 137.75) (size 2.2) (drill 2.1) (layers F.Cu B.Cu) (net 2))
@@
   (segment (start 153.5 122.5) (end 153.5 121.5) (width 0.5) (layer F.Cu) (net 39))
   (segment (start 153 123) (end 153.5 122.5) (width 0.5) (layer F.Cu) (net 39))
+  (via (at 113.5 117.5) (size 0.8) (drill 0.4) (layers F.Cu B.Cu) (net 39))
+  (segment (start 109.13 117.5) (end 113.5 117.5) (width 0.5) (layer F.Cu) (net 39))
+  (segment (start 101.88 110.25) (end 109.13 117.5) (width 0.5) (layer F.Cu) (net 39))
+  (via (at 113.5 108.75) (size 0.8) (drill 0.4) (layers F.Cu B.Cu) (net 39))
+  (segment (start 113.5 117.5) (end 113.5 108.75) (width 0.5) (layer B.Cu) (net 39))
+  (segment (start 113.5 108.75) (end 133.5 108.75) (width 0.5) (layer F.Cu) (net 39))
+  (via (at 136.75 111.717999) (size 0.8) (drill 0.4) (layers F.Cu B.Cu) (net 39))
+  (segment (start 136.158001 110.399999) (end 136.75 110.991998) (width 0.5) (layer F.Cu) (net 39))
+  (segment (start 135.149999 110.399999) (end 136.158001 110.399999) (width 0.5) (layer F.Cu) (net 39))
+  (segment (start 136.75 110.991998) (end 136.75 111.717999) (width 0.5) (layer F.Cu) (net 39))
+  (segment (start 133.5 108.75) (end 135.149999 110.399999) (width 0.5) (layer F.Cu) (net 39))
+  (segment (start 136.75 111.717999) (end 142.217999 111.717999) (width 0.5) (layer B.Cu) (net 39))
+  (segment (start 142.217999 110.322001) (end 142.25 110.29) (width 0.5) (layer B.Cu) (net 39))
+  (segment (start 142.217999 111.717999) (end 142.217999 110.322001) (width 0.5) (layer B.Cu) (net 39))
   (segment (start 143.550001 106.449999) (end 142.25 107.75) (width 0.5) (layer F.Cu) (net 40))
   (segment (start 150.494001 106.449999) (end 143.550001 106.449999) (width 0.5) (layer F.Cu) (net 40))

Commit message: Current board designs
Routing:
- net +5V: track 0.00 -> 36.9 mm
