File: teabiscuits_integween/teabiscuits_compute.sch (KiCad schematic (older format))
At the start: 17 parts, among them J2 Conn_02x05_Odd_Even, J3 Conn_01x03, J4 Conn_02x05_Odd_Even, J5 Conn_02x03_Odd_Even, J6 J1B1211CCD, U1 teensy41, U2 PDME1-S5-D3-S, U3 ADP7142AUJZ-2.5, U4 ADP7182AUJZ-2.5, U5 REF5020AD

Commit message: integween r9
Changed lines of the file:
@@
 DAC_LDAC
 $Comp
-L power:+5V #PWR0101
-U 1 1 5F4D6676
+L power:+2V5 #PWR?
+U 1 1 5FA488E0
 P 1350 1250
-F 0 "#PWR0101" H 1350 1100 50  0001 C CNN
-F 1 "+5V" V 1350 1450 50  0000 C CNN
+F 0 "#PWR?" H 1350 1100 50  0001 C CNN
+F 1 "+2V5" V 1350 1450 50  0000 C CNN
 F 2 "" H 1350 1250 50  0001 C CNN
 F 3 "" H 1350 1250 50  0001 C CNN

Commit message: Current board designs
Parts:
- C5: value 0.1uF -> 1uF
- C6: value 0.1uF -> 22uF
- U1: symbol teensy41:teensy41 -> teabiscuits_compute-rescue:teensy41-teensy41
- U4: symbol Regulator_Linear:ADP7182AUJZ-2.5 -> teabiscuits_compute-rescue:ADP7182AUJZ-2.5-Regulator_Linear
Changed lines of the file:
@@
 SPI1_SCLK
 $Comp
-L teensy41:teensy41 U1
+L teabiscuits_compute-rescue:teensy41-teensy41 U1
 U 1 1 5F2E3EA3
 P 1900 5750
@@
 $EndComp
 $Comp
-L Regulator_Linear:ADP7182AUJZ-2.5 U4
+L teabiscuits_compute-rescue:ADP7182AUJZ-2.5-Regulator_Linear U4
 U 1 1 5F94E553
 P 3650 4000
@@
 P 7550 3700
 F 0 "C6" H 7665 3746 50  0000 L CNN
-F 1 "0.1uF" H 7665 3655 50  0000 L CNN
+F 1 "22uF" H 7665 3655 50  0000 L CNN
 F 2 "Capacitor_SMD:C_0805_2012Metric" H 7588 3550 50  0001 C CNN
 F 3 "~" H 7550 3700 50  0001 C CNN
@@
 P 6650 3050
 F 0 "C5" V 6398 3050 50  0000 C CNN
-F 1 "0.1uF" V 6489 3050 50  0000 C CNN
+F 1 "1uF" V 6489 3050 50  0000 C CNN
 F 2 "Capacitor_SMD:C_0805_2012Metric" H 6688 2900 50  0001 C CNN
 F 3 "~" H 6650 3050 50  0001 C CNN
